File: madeline36/pcb/madeline36-pcb.kicad_pcb (KiCad board)
At the start: 2 copper layers, 234.2 x 93.1 mm, 78 parts, among them SW1 SW_SPST, SW10 SW_SPST, SW11 SW_SPST, SW12 SW_SPST, SW13 SW_SPST, SW14 SW_SPST, SW15 SW_SPST, SW16 SW_SPST, SW17 SW_SPST, SW18 SW_SPST, SW19 SW_SPST, SW2 SW_SPST, SW20 SW_SPST, SW21 SW_SPST, SW22 SW_SPST, SW23 SW_SPST, SW24 SW_SPST, SW25 SW_SPST, SW26 SW_SPST, SW27 SW_SPST, SW28 SW_SPST, SW29 SW_SPST, SW3 SW_SPST, SW30 SW_SPST, SW31 SW_SPST, SW32 SW_SPST, SW33 SW_SPST, SW34 SW_SPST, SW35 SW_SPST, SW36 SW_SPST, SW4 SW_SPST, SW5 SW_SPST, SW6 SW_SPST, SW7 SW_SPST, SW8 SW_SPST, SW9 SW_SPST, U1 rp2040-zero

Commit message: dim. 10 mars 2024 23:07:29 CET
Routing:
- net c0: track 337.0 -> 340.2 mm
- net l3: track 140.7 -> 142.2 mm
Changed lines of the file:
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@@
   (segment (start 139.7737 178.4083) (end 138.2655 178.1424) (width 0.4) (layer "F.Cu") (net 37))
   (segment (start 114.25 175.889) (end 136.0121 175.889) (width 0.4) (layer "F.Cu") (net 37))
-  (segment (start 197.0746 174.7137) (end 197.0746 165.5658) (width 0.4) (layer "B.Cu") (net 37))
-  (segment (start 197.0746 165.5658) (end 200.0772 162.5632) (width 0.4) (layer "B.Cu") (net 37))
-  (segment (start 201.3291 133.1189) (end 200.0772 133.1189) (width 0.4) (layer "B.Cu") (net 37))
+  (segment (start 204.046875 158.334375) (end 200.0772 154.3647) (width 0.4) (layer "B.Cu") (net 37))
   (segment (start 141.2819 178.6742) (end 139.7737 178.4083) (width 0.4) (layer "B.Cu") (net 37))
-  (segment (start 200.0772 162.5632) (end 200.0772 134.8893) (width 0.4) (layer "B.Cu") (net 37))
-  (segment (start 200.0772 134.8893) (end 201.3291 133.6374) (width 0.4) (layer "B.Cu") (net 37))
-  (segment (start 181.4882 190.3001) (end 197.0746 174.7137) (width 0.4) (layer "B.Cu") (net 37))
+  (segment (start 181.4882 190.3001) (end 204.046875 167.741425) (width 0.4) (layer "B.Cu") (net 37))
+  (segment (start 204.046875 167.741425) (end 204.046875 158.334375) (width 0.4) (layer "B.Cu") (net 37))
+  (segment (start 200.0772 154.3647) (end 200.0772 133.1189) (width 0.4) (layer "B.Cu") (net 37))
   (segment (start 175.471875 191.671875) (end 154.279575 191.671875) (width 0.4) (layer "B.Cu") (net 37))
   (segment (start 181.4882 190.5261) (end 176.61765 190.5261) (width 0.4) (layer "B.Cu") (net 37))
   (segment (start 176.61765 190.5261) (end 175.471875 191.671875) (width 0.4) (layer "B.Cu") (net 37))
-  (segment (start 201.3291 133.6374) (end 201.3291 133.1189) (width 0.4) (layer "B.Cu") (net 37))
   (segment (start 154.279575 191.671875) (end 141.2819 178.6742) (width 0.4) (layer "B.Cu") (net 37))
   (segment (start 112.3777 167.6986) (end 112.9481 168.269) (width 0.4) (layer "F.Cu") (net 38))
@@
   (segment (start 200.475 136.903125) (end 189.41045 136.903125) (width 0.4) (layer "F.Cu") (net 45))
   (segment (start 111.4615 145.2375) (end 155.194899 145.2375) (width 0.4) (layer "F.Cu") (net 45))
-  (segment (start 202.6172 133.1189) (end 202.6172 123.667) (width 0.4) (layer "B.Cu") (net 45))
   (segment (start 104.3779 166.8217) (end 104.378 166.8217) (width 0.4) (layer "B.Cu") (net 45))
   (segment (start 309.0977 156.4508) (end 311.75 159.1031) (width 0.4) (layer "B.Cu") (net 45))
@@
   (segment (start 104.378 166.8217) (end 104.378 166.8218) (width 0.4) (layer "B.Cu") (net 45))
   (segment (start 308.065 150.159) (end 309.0977 151.1917) (width 0.4) (layer "B.Cu") (net 45))
+  (segment (start 211.194175 109.5152) (end 202.6172 118.092175) (width 0.4) (layer "B.Cu") (net 45))
   (segment (start 310.8 126.1861) (end 310.8 129.319) (width 0.4) (layer "B.Cu") (net 45))
+  (segment (start 202.6172 118.092175) (end 202.6172 133.1189) (width 0.4) (layer "B.Cu") (net 45))
+  (segment (start 302.3812 109.5152) (end 211.194175 109.5152) (width 0.4) (layer "B.Cu") (net 45))
   (segment (start 107.0448 150.5138) (end 107.0448 158.3139) (width 0.4) (layer "B.Cu") (net 45))
   (segment (start 107.0461 121.4506) (end 106.3711 120.7756) (width 0.4) (layer "B.Cu") (net 45))
-  (segment (start 302.3812 109.5152) (end 304.265 111.399) (width 0.4) (layer "B.Cu") (net 45))
   (segment (start 310.7919 140.8111) (end 310.7919 147.2821) (width 0.4) (layer "B.Cu") (net 45))
   (segment (start 304.8961 120.2822) (end 310.8 126.1861) (width 0.4) (layer "B.Cu") (net 45))
-  (segment (start 216.769 109.5152) (end 302.3812 109.5152) (width 0.4) (layer "B.Cu") (net 45))
   (segment (start 304.8961 112.0301) (end 304.8961 120.2822) (width 0.4) (layer "B.Cu") (net 45))
   (segment (start 106.3711 120.7756) (end 106.3711 112.0301) (width 0.4) (layer "B.Cu") (net 45))
   (segment (start 310.7919 147.2821) (end 309.375 148.699) (width 0.4) (layer "B.Cu") (net 45))
-  (segment (start 202.6172 123.667) (end 216.769 109.5152) (width 0.4) (layer "B.Cu") (net 45))
+  (segment (start 304.265 111.399) (end 302.3812 109.5152) (width 0.4) (layer "B.Cu") (net 45))
   (segment (start 190.411625 151.729) (end 205.1572 136.983425) (width 0.4) (layer "F.Cu") (net 46))
   (segment (start 159.6085 158.9664) (end 166.8459 151.729) (width 0.4) (layer "F.Cu") (net 46))
@@
     (connect_pads (clearance 0.5))
     (min_thickness 0.25) (filled_areas_thickness no)
-    (fill yes (thermal_gap 0.5) (thermal_bridge_width 0.5) (island_removal_mode 1) (island_area_min 10))
+    (fill yes (thermal_gap 0.5) (thermal_bridge_width 0.5))
     (polygon
       (pts
