File: split44/pcb/split44-pcb.kicad_pcb (KiCad board)
At the start: 2 copper layers, 146.2 x 111 mm, 53 parts, among them J1 AudioJack4, SW1 SW_SPST, SW10 SW_SPST, SW11 SW_SPST, SW12 SW_SPST, SW13 SW_SPST, SW14 SW_SPST, SW15 SW_SPST, SW16 SW_SPST, SW17 SW_SPST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

Commit message: ""
Parts:
- moved J1 4.76 mm to (283.0, 159.5)
Routing:
- net com_1: track 23.0 -> 44.6 mm, vias 0 -> 1
- net +5V: track 51.7 -> 71.6 mm
- net com_2: track 34.3 -> 16.7 mm, vias 1 -> 0
- net GND: track 18.2 -> 27.1 mm
- net l2: track 136.7 -> 137.7 mm
Changed lines of the file:
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@@
   )
   (footprint "lib:TRRS-PJ-320A_reversible" (layer "F.Cu")
-    (at 278.2656 159.525 -90)
+    (at 283.028125 159.525 -90)
     (property "Sheetfile" "split44-pcb.kicad_sch")
     (property "Sheetname" "")
@@
   (segment (start 238.4599 158.221) (end 222.3326 158.221) (width 0.4) (layer "F.Cu") (net 15))
   (segment (start 183.1252 169.7983) (end 183.1252 169.7984) (width 0.4) (layer "F.Cu") (net 15))
-  (segment (start 259.1418 150.1401) (end 264.3468 144.9351) (width 0.4) (layer "B.Cu") (net 15))
-  (segment (start 259.1418 158.4672) (end 259.1418 150.1401) (width 0.4) (layer "B.Cu") (net 15))
-  (segment (start 263.314875 135.8712) (end 264.3468 136.903125) (width 0.4) (layer "B.Cu") (net 15))
-  (segment (start 257.8399 161.071) (end 257.8399 159.7691) (width 0.4) (layer "B.Cu") (net 15))
+  (segment (start 261.196875 148.085025) (end 264.3468 144.9351) (width 0.4) (layer "B.Cu") (net 15))
   (segment (start 264.3468 144.9351) (end 264.3468 136.903125) (width 0.4) (layer "B.Cu") (net 15))
-  (segment (start 257.8399 159.7691) (end 259.1418 158.4672) (width 0.4) (layer "B.Cu") (net 15))
+  (segment (start 261.196875 159.525) (end 261.196875 148.085025) (width 0.4) (layer "B.Cu") (net 15))
+  (segment (start 264.3468 136.903125) (end 263.314875 135.8712) (width 0.4) (layer "B.Cu") (net 15))
+  (segment (start 259.650875 161.071) (end 261.196875 159.525) (width 0.4) (layer "B.Cu") (net 15))
+  (segment (start 257.8399 161.071) (end 259.650875 161.071) (width 0.4) (layer "B.Cu") (net 15))
   (segment (start 160.8142 168.8694) (end 158.6986 168.8694) (width 0.4) (layer "F.Cu") (net 16))
   (segment (start 160.8142 168.8695) (end 160.8142 168.8694) (width 0.4) (layer "F.Cu") (net 16))
@@
   (segment (start 262.50893 180.95625) (end 267.183605 185.630925) (width 0.4) (layer "F.Cu") (net 26))
   (segment (start 267.1836 190.0633) (end 267.1836 187.3987) (width 0.4) (layer "B.Cu") (net 26))
-  (segment (start 264.76875 157.14375) (end 263.578125 155.953125) (width 0.4) (layer "F.Cu") (net 27))
-  (segment (start 267.41245 157.14375) (end 264.76875 157.14375) (width 0.4) (layer "F.Cu") (net 27))
-  (segment (start 275.0656 156.724975) (end 274.023925 155.6833) (width 0.4) (layer "F.Cu") (net 27))
-  (segment (start 275.0656 159.525) (end 275.0656 156.724975) (width 0.4) (layer "F.Cu") (net 27))
-  (segment (start 263.578125 155.953125) (end 263.578125 153.699025) (width 0.4) (layer "F.Cu") (net 27))
-  (segment (start 263.5781 153.699) (end 263.5781 150.65) (width 0.4) (layer "F.Cu") (net 27))
-  (segment (start 274.023925 155.6833) (end 268.8729 155.6833) (width 0.4) (layer "F.Cu") (net 27))
-  (segment (start 268.8729 155.6833) (end 267.41245 157.14375) (width 0.4) (layer "F.Cu") (net 27))
-  (segment (start 263.578125 153.699025) (end 263.5781 153.699) (width 0.4) (layer "F.Cu") (net 27))
-  (segment (start 269.22375 166.66875) (end 264.76875 166.66875) (width 0.4) (layer "B.Cu") (net 27))
-  (segment (start 275.0656 160.8269) (end 269.22375 166.66875) (width 0.4) (layer "B.Cu") (net 27))
-  (segment (start 263.578125 161.906275) (end 263.5781 161.90625) (width 0.4) (layer "B.Cu") (net 27))
-  (segment (start 264.76875 166.66875) (end 263.578125 165.478125) (width 0.4) (layer "B.Cu") (net 27))
-  (segment (start 275.0656 159.525) (end 275.0656 160.8269) (width 0.4) (layer "B.Cu") (net 27))
-  (segment (start 263.5781 161.90625) (end 263.5781 150.65) (width 0.4) (layer "B.Cu") (net 27))
-  (segment (start 263.578125 165.478125) (end 263.578125 161.906275) (width 0.4) (layer "B.Cu") (net 27))
-  (segment (start 266.9656 154.925) (end 266.9656 150.8344) (width 0.4) (layer "F.Cu") (net 28))
-  (segment (start 266.9656 164.125) (end 265.959375 163.118775) (width 0.4) (layer "B.Cu") (net 28))
-  (segment (start 265.959375 157.233125) (end 266.9656 156.2269) (width 0.4) (layer "B.Cu") (net 28))
-  (segment (start 266.9656 156.2269) (end 266.9656 155.4999) (width 0.4) (layer "B.Cu") (net 28))
-  (segment (start 267.15 155.3155) (end 267.15 150.65) (width 0.4) (layer "B.Cu") (net 28))
-  (segment (start 265.959375 163.118775) (end 265.959375 157.233125) (width 0.4) (layer "B.Cu") (net 28))
+  (segment (start 277.865625 166.66875) (end 279.828125 164.70625) (width 0.4) (layer "F.Cu") (net 27))
+  (segment (start 279.828125 164.70625) (end 279.828125 159.525) (width 0.4) (layer "F.Cu") (net 27))
+  (segment (start 263.5781 164.287475) (end 265.959375 166.66875) (width 0.4) (layer "F.Cu") (net 27))
+  (segment (start 265.959375 166.66875) (end 277.865625 166.66875) (width 0.4) (layer "F.Cu") (net 27))
+  (segment (start 263.5781 150.65) (end 263.5781 164.287475) (width 0.4) (layer "F.Cu") (net 27))
+  (segment (start 263.5781 154.7625) (end 267.149975 158.334375) (width 0.4) (layer "B.Cu") (net 27))
+  (segment (start 267.15 158.334375) (end 267.15 164.2875) (width 0.4) (layer "B.Cu") (net 27))
+  (segment (start 267.15 164.2875) (end 269.53125 166.66875) (width 0.4) (layer "B.Cu") (net 27))
+  (segment (start 279.828125 159.525) (end 279.828125 164.70625) (width 0.4) (layer "B.Cu") (net 27))
+  (segment (start 279.828125 164.70625) (end 277.865625 166.66875) (width 0.4) (layer "B.Cu") (net 27))
+  (segment (start 277.865625 166.66875) (end 269.53125 166.66875) (width 0.4) (layer "B.Cu") (net 27))
+  (segment (start 263.5781 154.7625) (end 263.5781 150.65) (width 0.4) (layer "B.Cu") (net 27))
+  (segment (start 267.149975 158.334375) (end 267.15 158.334375) (width 0.4) (layer "B.Cu") (net 27))
+  (segment (start 267.15 153.571875) (end 267.15 150.65) (width 0.4) (layer "F.Cu") (net 28))
+  (segment (start 268.503125 154.925) (end 267.15 153.571875) (width 0.4) (layer "F.Cu") (net 28))
+  (segment (start 271.728125 154.925) (end 268.503125 154.925) (width 0.4) (layer "F.Cu") (net 28))
+  (segment (start 271.728125 154.946875) (end 269.53125 157.14375) (width 0.4) (layer "B.Cu") (net 28))
+  (segment (start 267.15 153.571875) (end 268.503125 154.925) (width 0.4) (layer "B.Cu") (net 28))
+  (segment (start 267.15 150.65) (end 267.15 153.571875) (width 0.4) (layer "B.Cu") (net 28))
+  (segment (start 269.53125 161.928125) (end 271.728125 164.125) (width 0.4) (layer "B.Cu") (net 28))
+  (segment (start 268.503125 154.925) (end 271.728125 154.925) (width 0.4) (layer "B.Cu") (net 28))
+  (segment (start 269.53125 157.14375) (end 269.53125 161.928125) (width 0.4) (layer "B.Cu") (net 28))
   (segment (start 263.6128 126.9812) (end 266.8868 130.2552) (width 0.4) (layer "B.Cu") (net 29))
   (segment (start 260.843 123.1712) (end 260.843 126.2564) (width 0.4) (layer "B.Cu") (net 29))
@@
   (segment (start 246.2999 152.181) (end 254.3204 144.1605) (width 0.4) (layer "B.Cu") (net 38))
   (segment (start 258.1525 144.1605) (end 261.3618 140.9512) (width 0.4) (layer "B.Cu") (net 38))
-  (segment (start 272.0656 164.4406) (end 274.29375 166.66875) (width 0.4) (layer "F.Cu") (net 40))
-  (segment (start 274.29375 166.66875) (end 276.675 166.66875) (width 0.4) (layer "F.Cu") (net 40))
-  (segment (start 272.0656 159.525) (end 272.0656 164.4406) (width 0.4) (layer "F.Cu") (net 40))
-  (via (at 276.675 166.66875) (size 0.6) (drill 0.3) (layers "F.Cu" "B.Cu") (net 40))
-  (segment (start 278.3349 143.4912) (end 278.3349 165.00885) (width 0.4) (layer "B.Cu") (net 40))
-  (segment (start 278.3349 165.00885) (end 276.675 166.66875) (width 0.4) (layer "B.Cu") (net 40))
-  (segment (start 261.196875 158.334375) (end 262.3875 159.525) (width 0.4) (layer "F.Cu") (net 46))
-  (segment (start 262.3875 159.525) (end 268.0656 159.525) (width 0.4) (layer "F.Cu") (net 46))
-  (segment (start 261.196875 145.389225) (end 261.196875 158.334375) (width 0.4) (layer "F.Cu") (net 46))
-  (segment (start 263.0949 143.4912) (end 261.196875 145.389225) (width 0.4) (layer "F.Cu") (net 46))
+  (segment (start 278.3349 143.4912) (end 278.3349 158.018225) (width 0.4) (layer "B.Cu") (net 40))
+  (segment (start 278.3349 158.018225) (end 276.828125 159.525) (width 0.4) (layer "B.Cu") (net 40))
+  (segment (start 272.828125 159.525) (end 264.76875 159.525) (width 0.4) (layer "F.Cu") (net 46))
+  (via (at 264.76875 159.525) (size 0.6) (drill 0.3) (layers "F.Cu" "B.Cu") (net 46))
+  (segment (start 255.24375 164.2875) (end 255.24375 151.34235) (width 0.4) (layer "B.Cu") (net 46))
+  (segment (start 255.24375 164.2875) (end 256.434375 165.478125) (width 0.4) (layer "B.Cu") (net 46))
+  (segment (start 255.24375 151.34235) (end 263.0949 143.4912) (width 0.4) (layer "B.Cu") (net 46))
+  (segment (start 258.815625 165.478125) (end 256.434375 165.478125) (width 0.4) (layer "B.Cu") (net 46))
+  (segment (start 264.76875 159.525) (end 258.815625 165.478125) (width 0.4) (layer "B.Cu") (net 46))
   (zone (net 0) (net_name "") (layers "F&B.Cu") (hatch edge 0.5)
     (connect_pads (clearance 0.5))
