File: split46/pcb/split46-pcb.kicad_pcb (KiCad board)
At the start: 2 copper layers, 136.6 x 94.6 mm, 55 parts, among them J1 AudioJack4, SW1 SW_SPST, SW10 SW_SPST, SW11 SW_SPST, SW12 SW_SPST, SW13 SW_SPST, SW14 SW_SPST, SW15 SW_SPST, SW16 SW_SPST, SW17 SW_SPST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

Commit message: dim. 17 mars 2024 09:56:18 CET
Connections:
- J1 pad R1: unconnected-(J1-PadR1) -> com_1
- J1 pad R2: unconnected-(J1-PadR2) -> com_2
Routing:
- net com_1: track 0.00 -> 39.0 mm
- net com_2: track 0.00 -> 34.3 mm
- net GND: track 24.8 -> 29.0 mm

Commit message: ""
Parts:
- U1: footprint mcu:rp2040-zero-tht -> _mcu:rp2040-zero-tht
- moved J1 4.68 mm to (280.2, 153.8)
Routing:
- net com_1: track 39.0 -> 21.8 mm
- net +5V: track 33.5 -> 48.7 mm
- net com_2: track 34.3 -> 20.7 mm
- net c3: track 148.3 -> 138.8 mm
- net c1: track 189.8 -> 180.9 mm
- net GND: track 29.0 -> 21.8 mm
- net c2: track 140.5 -> 134.0 mm
- net c4: track 134.4 -> 128.0 mm
- net c5: track 92.5 -> 86.2 mm
- net c0: track 202.1 -> 195.9 mm
- net Net-(D6-A): track 17.5 -> 14.2 mm
- net Net-(D18-A): track 17.6 -> 14.3 mm
- net Net-(D12-A): track 17.5 -> 14.3 mm
- net Net-(D5-A): track 10.2 -> 8.23 mm
- net Net-(D13-A): track 9.99 -> 8.00 mm
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