File: classic/simple51/pcb/simple51.kicad_pcb (KiCad board)
At the start: 2 copper layers, 245.3 x 102.4 mm, 108 parts, among them SW1 SW_SPST, SW10 SW_SPST, SW11 SW_SPST, SW12 SW_SPST, SW13 SW_SPST, SW14 SW_SPST, SW15 SW_SPST, SW16 SW_SPST, SW17 SW_SPST, SW18 SW_SPST, SW19 SW_SPST, SW2 SW_SPST, SW20 SW_SPST, SW21 SW_SPST, SW22 SW_SPST, SW23 SW_SPST, SW24 SW_SPST, SW25 SW_SPST, SW26 SW_SPST, SW27 SW_SPST, SW28 SW_SPST, SW29 SW_SPST, SW3 SW_SPST, SW30 SW_SPST, SW31 SW_SPST, SW32 SW_SPST, SW33 SW_SPST, SW34 SW_SPST, SW35 SW_SPST, SW36 SW_SPST, SW37 SW_SPST, SW38 SW_SPST, SW39 SW_SPST, SW4 SW_SPST, SW40 SW_SPST, SW41 SW_SPST, SW42 SW_SPST, SW43 SW_SPST, SW44 SW_SPST, SW45 SW_SPST, SW46 SW_SPST, SW47 SW_SPST, SW48 SW_SPST, SW49 SW_SPST, SW5 SW_SPST, SW50 SW_SPST, SW51 SW_SPST, SW6 SW_SPST, SW7 SW_SPST, SW8 SW_SPST, SW9 SW_SPST, U1 rp2040-zero

Commit message: sam. 13 juil. 2024 16:38:29 CEST
Parts:
- moved D17 9.53 mm to (282.6, 127.1)
- moved D40 9.53 mm to (277.9, 165.2)
- moved D49 9.53 mm to (277.9, 184.3)
- moved SW17 9.53 mm to (288.4, 136.0)
- moved SW40 9.53 mm to (283.7, 174.1)
- moved SW49 9.53 mm to (283.7, 193.2)
- moved D1 9.53 mm to (101.7, 103.3)
- moved D11 9.53 mm to (168.3, 127.1)
- moved D12 9.53 mm to (187.4, 127.1)
- moved D13 9.53 mm to (206.4, 127.1)
- moved D14 9.53 mm to (225.5, 127.1)
- moved D16 9.53 mm to (263.6, 127.1)
- moved D2 9.53 mm to (120.7, 103.3)
- moved D22 9.53 mm to (154.0, 146.2)
- moved D24 9.53 mm to (192.1, 146.2)
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Other:
- outline, holes or cut-outs redrawn
- board text added: "simple51"
