File: ergo/ergo47/pcb/ergo47.kicad_pcb (KiCad board)
At the start: 2 copper layers, 274.6 x 114.7 mm, 108 parts, among them SW1 SW_SPST, SW10 SW_SPST, SW11 SW_SPST, SW12 SW_SPST, SW13 SW_SPST, SW14 SW_SPST, SW15 SW_SPST, SW16 SW_SPST, SW17 SW_SPST, SW18 SW_SPST, SW19 SW_SPST, SW2 SW_SPST, SW20 SW_SPST, SW21 SW_SPST, SW22 SW_SPST, SW23 SW_SPST, SW24 SW_SPST, SW25 SW_SPST, SW26 SW_SPST, SW27 SW_SPST, SW28 SW_SPST, SW29 SW_SPST, SW3 SW_SPST, SW30 SW_SPST, SW31 SW_SPST, SW32 SW_SPST, SW33 SW_SPST, SW34 SW_SPST, SW35 SW_SPST, SW36 SW_SPST, SW37 SW_SPST, SW38 SW_SPST, SW39 SW_SPST, SW4 SW_SPST, SW40 SW_SPST, SW41 SW_SPST, SW42 SW_SPST, SW43 SW_SPST, SW44 SW_SPST, SW45 SW_SPST, SW46 SW_SPST, SW47 SW_SPST, SW5 SW_SPST, SW6 SW_SPST, SW7 SW_SPST, SW8 SW_SPST, SW9 SW_SPST, U1 rp2040-zero

Commit message: lun. 15 juil. 2024 17:34:45 CEST
Parts:
- removed STAB01: Stabilizer_Cherry_MX_2.00u, _mx:Stabilizer_Cherry_MX_2.00u
- REF01: renamed from REF02; value MountingHole_2.2mm_M2 -> MountingHole
- REF02: renamed from REF13; value MountingHole_2.2mm_M2 -> MountingHole
- REF03, REF04, REF05, REF06, REF07, REF08, REF09, REF10, REF11, REF12: value MountingHole_2.2mm_M2 -> MountingHole
- SW41: footprint _mx:SW_Cherry_MX_PCB -> _mx:SW_Cherry_MX_PCB_2.00u
- U1: moved to B.Cu
- moved D42 31.3 mm to (180.2, 176.5), turned to 75 degrees
- moved D41 24.3 mm to (186.8, 178.3), turned to 75 degrees
- moved D40 3.00 mm to (177.1, 175.7)
- turned SW41 to 180 degrees
- turned U1 to -105 degrees
Connections:
- U1 pad 1: unconnected-(U1-Pad1) -> C1
- U1 pad 10: L4 -> L3
- U1 pad 11: L3 -> L4
- U1 pad 12: L2 -> L5
- U1 pad 13: L1 -> L6
- U1 pad 14: C6 -> L7
- U1 pad 15: C5 -> L8
- U1 pad 16: C4 -> unconnected-(U1-Pad16)
- U1 pad 17: C3 -> unconnected-(U1-Pad17)
- U1 pad 18: C2 -> unconnected-(U1-Pad18)
- U1 pad 19: C1 -> unconnected-(U1-Pad19)
- U1 pad 2: unconnected-(U1-Pad2) -> C2
- U1 pad 3: unconnected-(U1-Pad3) -> C3
- U1 pad 4: unconnected-(U1-Pad4) -> C4
- U1 pad 5: unconnected-(U1-Pad5) -> C5
- U1 pad 6: L8 -> C6
- U1 pad 7: L7 -> unconnected-(U1-Pad7)
- U1 pad 8: L6 -> L1
- U1 pad 9: L5 -> L2
Routing:
- net C4: track 299.0 -> 388.2 mm
- net L8: track 145.3 -> 200.0 mm, vias 1 -> 0
- net L7: track 169.1 -> 210.7 mm, vias 1 -> 0
- net C6: track 194.6 -> 157.8 mm
- net C5: track 271.7 -> 308.1 mm
- net Net-(D42-Pad2): track 14.5 -> 49.7 mm
- net C2: track 446.0 -> 461.4 mm
- net Net-(D41-Pad2): track 10.3 -> 25.3 mm
- net L2: track 170.5 -> 161.6 mm
- net L3: track 193.9 -> 187.2 mm
- net L6: track 182.1 -> 188.3 mm
- net L1: track 145.0 -> 140.7 mm
- net Net-(D40-Pad2): track 6.94 -> 10.3 mm
- net C3: track 387.7 -> 389.8 mm, vias 0 -> 2
- net L4: track 226.1 -> 224.3 mm, vias 1 -> 0
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Other:
- outline, holes or cut-outs redrawn
