File: ergo/ergo47/pcb/ergo47.kicad_sch (KiCad schematic)
At the start: 95 parts, among them SW1 SW_SPST, SW10 SW_SPST, SW11 SW_SPST, SW12 SW_SPST, SW13 SW_SPST, SW14 SW_SPST, SW15 SW_SPST, SW16 SW_SPST, SW17 SW_SPST, SW18 SW_SPST, SW19 SW_SPST, SW2 SW_SPST, SW20 SW_SPST, SW21 SW_SPST, SW22 SW_SPST, SW23 SW_SPST, SW24 SW_SPST, SW25 SW_SPST, SW26 SW_SPST, SW27 SW_SPST, SW28 SW_SPST, SW29 SW_SPST, SW3 SW_SPST, SW30 SW_SPST, SW31 SW_SPST, SW32 SW_SPST, SW33 SW_SPST, SW34 SW_SPST, SW35 SW_SPST, SW36 SW_SPST, SW37 SW_SPST, SW38 SW_SPST, SW39 SW_SPST, SW4 SW_SPST, SW40 SW_SPST, SW41 SW_SPST, SW42 SW_SPST, SW43 SW_SPST, SW44 SW_SPST, SW45 SW_SPST, SW46 SW_SPST, SW47 SW_SPST, SW5 SW_SPST, SW6 SW_SPST, SW7 SW_SPST, SW8 SW_SPST, SW9 SW_SPST, U1 rp2040-zero

Commit message: lun. 15 juil. 2024 17:34:45 CEST
Parts:
- added REF01, REF02, REF03, REF04, REF05, REF06, REF07, REF08, REF09, REF10, REF11, REF12: MountingHole, MountingHole:MountingHole_2.2mm_M2, symbol Mechanical:MountingHole
- SW41: footprint _mx:SW_Cherry_MX_PCB -> _mx:SW_Cherry_MX_PCB_2.00u
Connections:
- net C1: now also U1.1 (0); no longer U1.19 (28)
- net C2: now also U1.2 (1); no longer U1.18 (27)
- net C3: now also U1.3 (2); no longer U1.17 (26)
- net C4: now also U1.4 (3); no longer U1.16 (15)
- net C5: now also U1.5 (4); no longer U1.15 (14)
- net C6: now also U1.6 (5); no longer U1.14 (13)
- net L1: now also U1.8 (7); no longer U1.13 (12)
- net L2: now also U1.9 (8); no longer U1.12 (11)
- net L3: now also U1.10 (9); no longer U1.11 (10)
- net L4: now also U1.11 (10); no longer U1.10 (9)
- net L5: now also U1.12 (11); no longer U1.9 (8)
- net L6: now also U1.13 (12); no longer U1.8 (7)
- net L7: now also U1.14 (13); no longer U1.7 (6)
- net L8: now also U1.15 (14); no longer U1.6 (5)
