File: classic/s45/s45.kicad_pcb (KiCad board)
At the start: 2 copper layers, 242.2 x 76 mm, 96 parts, among them SW1 key, SW10 key, SW11 key, SW12 key, SW13 key, SW14 key, SW15 key, SW16 key, SW17 key, SW18 key, SW19 key, SW2 key, SW20 key, SW21 key, SW22 key, SW23 key, SW24 key, SW25 key, SW26 key, SW27 key, SW28 key, SW29 key, SW3 key, SW30 key, SW31 key, SW32 key, SW33 key, SW34 key, SW35 key, SW36 key, SW37 key, SW38 key, SW39 key, SW4 key, SW40 key, SW41 key, SW42 key, SW43 key, SW44 key, SW45 key, SW5 key, SW6 key, SW7 key, SW8 key, SW9 key, U1 RP2040

Commit message: sam. 19 oct. 2024 18:38:35 CEST
Parts:
- turned SW21 to 0 degrees
Connections:
- SW21 pad 1: c8 -> Net-(D21-Pad2)
- SW21 pad 2: Net-(D21-Pad2) -> c8
Routing:
- net Net-(D21-Pad2): track 26.5 -> 18.0 mm
- net c8: track 83.4 -> 82.1 mm
Changed lines of the file:
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@@
   )
   (footprint "keyb-libs:MX-5pin" (layer "F.Cu")
-    (at 195.125 90.5 -90)
+    (at 195.125 90.5)
     (property "Sheetfile" "s45.kicad_sch")
     (property "Sheetname" "")
     (attr through_hole)
-    (fp_text reference "SW21" (at 0 5.08 -90 unlocked) (layer "F.SilkS") hide
+    (fp_text reference "SW21" (at 0 5.08 unlocked) (layer "F.SilkS") hide
       (effects (font (size 2 2) (thickness 0.15)))
     )
-    (fp_text value "key" (at 3.81 6.35 -90 unlocked) (layer "F.Fab") hide
+    (fp_text value "key" (at 3.81 6.35 unlocked) (layer "F.Fab") hide
       (effects (font (size 1 1) (thickness 0.15)))
     )
-    (fp_text user "${REFERENCE}" (at -3.81 -5.08 -90 unlocked) (layer "F.Fab") hide
+    (fp_text user "${REFERENCE}" (at -3.81 -5.08 unlocked) (layer "F.Fab") hide
       (effects (font (size 1 1) (thickness 0.15)))
     )
     (fp_rect (start -7 -7) (end 7 7) (layer "F.SilkS") (width 0.05) (fill none))
-    (pad "" np_thru_hole circle (at 5.08 0 270) (size 1.7 1.7) (drill 1.7) (layers *.Cu *.Mask))
-    (pad "" np_thru_hole circle (at 0 0 270) (size 4 4) (drill 4) (layers *.Cu *.Mask))
-    (pad "" np_thru_hole circle (at -5.08 0 270) (size 1.7 1.7) (drill 1.7) (layers *.Cu *.Mask))
-    (pad "1" thru_hole circle (at -3.81 -2.54 270) (size 2.4 2.4) (drill 1.5) (layers *.Cu *.Mask)
-      (net 58 "c8") (pinfunction "1") (pintype "bidirectional"))
-    (pad "2" thru_hole circle (at 2.54 -5.08 270) (size 2.4 2.4) (drill 1.5) (layers *.Cu *.Mask)
-      (net 23 "Net-(D21-Pad2)") (pinfunction "2") (pintype "bidirectional"))
+    (pad "" np_thru_hole circle (at 5.08 0) (size 1.7 1.7) (drill 1.7) (layers *.Cu *.Mask))
+    (pad "" np_thru_hole circle (at 0 0) (size 4 4) (drill 4) (layers *.Cu *.Mask))
+    (pad "" np_thru_hole circle (at -5.08 0) (size 1.7 1.7) (drill 1.7) (layers *.Cu *.Mask))
+    (pad "1" thru_hole circle (at -3.81 -2.54) (size 2.4 2.4) (drill 1.5) (layers *.Cu *.Mask)
+      (net 23 "Net-(D21-Pad2)") (pinfunction "1") (pintype "bidirectional"))
+    (pad "2" thru_hole circle (at 2.54 -5.08) (size 2.4 2.4) (drill 1.5) (layers *.Cu *.Mask)
+      (net 58 "c8") (pinfunction "2") (pintype "bidirectional"))
     (model "${KIPRJMOD}/switch.step"
       (offset (xyz 0 -1 4.5))
@@
   (segment (start 175.185 80.5) (end 175.185 81.9519) (width 0.5) (layer "B.Cu") (net 22))
   (segment (start 175.1969 81.9519) (end 178.665 85.42) (width 0.5) (layer "B.Cu") (net 22))
-  (segment (start 181.75 93.015) (end 181.775 93.04) (width 0.5) (layer "B.Cu") (net 23))
-  (segment (start 179.21 100) (end 179.21 95.555) (width 0.5) (layer "B.Cu") (net 23))
-  (segment (start 181.775 93.04) (end 200.205 93.04) (width 0.5) (layer "B.Cu") (net 23))
-  (segment (start 179.21 95.555) (end 181.75 93.015) (width 0.5) (layer "B.Cu") (net 23))
+  (segment (start 179.21 98.367944) (end 179.21 100) (width 0.5) (layer "B.Cu") (net 23))
+  (segment (start 191.315 87.96) (end 189.617944 87.96) (width 0.5) (layer "B.Cu") (net 23))
+  (segment (start 189.617944 87.96) (end 179.21 98.367944) (width 0.5) (layer "B.Cu") (net 23))
   (segment (start 224.125 86.69) (end 217.935 86.69) (width 0.5) (layer "F.Cu") (net 24))
   (segment (start 217.935 86.69) (end 216.665 85.42) (width 0.5) (layer "F.Cu") (net 24))
@@
   (segment (start 169.94 125.96) (end 169.94 123.5661) (width 0.5) (layer "B.Cu") (net 56))
   (segment (start 163.2719 107.4169) (end 162.815 106.96) (width 0.5) (layer "B.Cu") (net 56))
-  (segment (start 172.315 87.96) (end 190.67581 87.96) (width 0.5) (layer "F.Cu") (net 57))
   (segment (start 198.3317 125.96) (end 182.2719 109.9002) (width 0.5) (layer "F.Cu") (net 57))
-  (segment (start 190.67581 87.96) (end 195.125 83.51081) (width 0.5) (layer "F.Cu") (net 57))
+  (segment (start 193.942 85.522) (end 195.125 84.339) (width 0.5) (layer "F.Cu") (net 57))
+  (segment (start 182.868 87.96) (end 185.306 85.522) (width 0.5) (layer "F.Cu") (net 57))
+  (segment (start 185.306 85.522) (end 193.942 85.522) (width 0.5) (layer "F.Cu") (net 57))
   (segment (start 200.815 125.96) (end 198.3317 125.96) (width 0.5) (layer "F.Cu") (net 57))
   (segment (start 182.2719 107.4169) (end 181.815 106.96) (width 0.5) (layer "F.Cu") (net 57))
-  (segment (start 195.125 83.51081) (end 195.125 82.88) (width 0.5) (layer "F.Cu") (net 57))
+  (segment (start 172.315 87.96) (end 182.868 87.96) (width 0.5) (layer "F.Cu") (net 57))
   (segment (start 182.2719 109.9002) (end 182.2719 107.4169) (width 0.5) (layer "F.Cu") (net 57))
+  (segment (start 195.125 84.339) (end 195.125 82.88) (width 0.5) (layer "F.Cu") (net 57))
   (segment (start 181.815 106.96) (end 181.586 106.731) (width 0.5) (layer "B.Cu") (net 57))
   (segment (start 174.175 100.553) (end 174.175 93.3634) (width 0.5) (layer "B.Cu") (net 57))
@@
   (segment (start 167.565 68.96) (end 168.0218 69.4168) (width 0.5) (layer "B.Cu") (net 57))
   (segment (start 168.0218 78.3222) (end 172.315 82.6154) (width 0.5) (layer "B.Cu") (net 57))
+  (segment (start 197.665 82.88) (end 197.665 85.42) (width 0.5) (layer "F.Cu") (net 58))
   (segment (start 179.21 88.57) (end 181.75 86.03) (width 0.5) (layer "B.Cu") (net 58))
   (segment (start 198.641 102.159) (end 178.321 102.159) (width 0.5) (layer "B.Cu") (net 58))
@@
   (segment (start 186.565 68.96) (end 187.465 69.86) (width 0.5) (layer "B.Cu") (net 58))
   (segment (start 186.195 75.87) (end 193.18 75.87) (width 0.5) (layer "B.Cu") (net 58))
-  (segment (start 197.665 86.69) (end 197.665 82.88) (width 0.5) (layer "B.Cu") (net 58))
   (segment (start 177.305 94.285) (end 179.21 92.38) (width 0.5) (layer "B.Cu") (net 58))
   (segment (start 187.465 69.86) (end 187.465 75.87) (width 0.5) (layer "B.Cu") (net 58))
